Commit message: reward tuning

File: simple_rexy/resources/simplegoal.urdf (robot description, URDF)
Before this commit: robot simplegoal, 1 links, 0 joints
Links:
- link base_link: geometry collision cylinder length=0.5 radius=0.25; visual cylinder length=.25 radius=0.25

File: simple_rexy/resources/simpleplane.urdf (robot description, URDF)
Before this commit: robot simpleplane, 1 links, 0 joints
Links:
- link base_link: geometry collision box size=7 5 0.01; visual box size=7 5 0.01
